Commit message: Renamed urdf file and updated launch files accordingly

File: phoebe_description/urdf/phoebe.urdf.xacro (robot description, xacro)
@@ -2,7 +2,7 @@
 <robot xmlns:xacro="http://www.ros.org/wiki/xacro" name="phoebe">
  <!-- <xacro:include filename="$(find cyton_gamma_1500_minicam_description)/cyton_gamma_1500_minicam_macros.urdf.xacro" /> -->
-  <xacro:include filename="$(find control_test)/urdf/cyton_gamma_1500_macros.urdf.xacro" />
+  <xacro:include filename="$(find cyton_gamma_1500_description)/urdf/cyton_gamma_1500_macros.urdf.xacro" />
   <xacro:include filename="$(find dp_ptu_46_description)/dp_ptu_46_macros.urdf.xacro" />
-  <xacro:include filename="$(find phoebe_description)/phoebe.gazebo" />
+  <xacro:include filename="$(find phoebe_description)/urdf/phoebe.gazebo" />
   <link name="base_footprint"/>
   <joint name="base_joint" type="fixed">
@@ -42,5 +42,5 @@
     <inertial>
       <!--origin rpy="0 0 0" xyz="0 0 0"/-->
-	  <origin rpy="0 1.5707 1.5707" xyz="0 0 0"/>
+	  <origin rpy="0 1.5708 1.5708" xyz="0 0 0"/>
       <mass value="0.25"/>
       <!-- inretia tensor for solid cylinder: m=0.5, h=0.05, r=0.095 -->
@@ -50,5 +50,5 @@
       <origin rpy="0 1.5707 1.5707" xyz="0 0 0"/>
       <geometry>
-        <cylinder length="0.04" radius="0.02"/>
+        <cylinder length="0.1" radius="0.02"/>
       </geometry>
       <material name="blackish">
@@ -59,5 +59,5 @@
       <origin rpy="0 1.5707 1.5707" xyz="0 0 0"/>
       <geometry>
-        <cylinder length="0.04" radius="0.02"/>
+        <cylinder length="0.1" radius="0.02"/>
       </geometry>
     </collision>
@@ -74,5 +74,5 @@
     <inertial>
       <!--origin rpy="0 0 0" xyz="0 0 0"/-->
-	  <origin rpy="0 1.5707 1.5707" xyz="0 0 0"/>
+	  <origin rpy="0 1.5708 1.5708" xyz="0 0 0"/>
       <mass value="0.25"/>
       <inertia ixx="1.232291667e-03" ixy="0" ixz="0" iyy="1.232291667e-03" iyz="0" izz="2.25625e-03"/>
@@ -81,5 +81,5 @@
      <origin rpy="0 1.5707 1.5707" xyz="0 0 0"/>
      <geometry>
-        <cylinder length="0.04" radius="0.02"/>
+        <cylinder length="0.1" radius="0.02"/>
       </geometry>
       <material name="blackish"/>
@@ -88,5 +88,5 @@
       <origin rpy="0 1.5707 1.5707" xyz="0 0 0"/>
       <geometry>
-        <cylinder length="0.04" radius="0.02"/>
+        <cylinder length="0.1" radius="0.02"/>
       </geometry>
     </collision>
@@ -99,9 +99,11 @@
     <!--axis xyz="0 0 1"/-->
 	<axis xyz="0 1 0"/>
+	<limit effort="10000" velocity="1000"/>
+    <joint_properties damping="1.0" friction="1.0"/>
   </joint>
   <link name="wheel_left">
     <inertial>
       <!--origin rpy="0 0 0" xyz="0 0 0"/-->
-	  <origin rpy="0 1.5707 1.5707" xyz="0 0 0"/>
+	  <origin rpy="0 1.5708 1.5708" xyz="0 0 0"/>
       <mass value="0.5"/>
       <!-- inretia tensor for solid cylinder: m=0.5, h=0.05, r=0.095 -->
@@ -110,5 +112,5 @@
     <visual>
       <!--origin rpy="0 0 0" xyz="0 0 0"/-->
-	  <origin rpy="0 1.5707 1.5707" xyz="0 0 0"/>
+	  <origin rpy="0 1.5708 1.5708" xyz="0 0 0"/>
       <geometry>
         <cylinder length="0.05" radius="0.095"/>
@@ -133,9 +135,11 @@
     <!--axis xyz="0 0 1"/-->
 	<axis xyz="0 1 0"/>
+	<limit effort="10000" velocity="1000"/>
+    <joint_properties damping="1.0" friction="1.0"/>
   </joint>
   <link name="wheel_right">
     <inertial>
       <!--origin rpy="0 0 0" xyz="0 0 0"/-->
-	  <origin rpy="0 1.5707 1.5707" xyz="0 0 0"/>
+	  <origin rpy="0 1.5708 1.5708" xyz="0 0 0"/>
       <mass value="0.5"/>
       <!-- inretia tensor for solid cylinder: m=0.5, h=0.05, r=0.095 -->
@@ -144,5 +148,5 @@
     <visual>
       <!--origin rpy="0 0 0" xyz="0 0 0"/-->
-	  <origin rpy="0 1.5707 1.5707" xyz="0 0 0"/>
+	  <origin rpy="0 1.5708 1.5708" xyz="0 0 0"/>
       <geometry>
         <cylinder length="0.05" radius="0.095"/>
@@ -152,5 +156,5 @@
     <collision>
       <!--origin rpy="0 0 0" xyz="0 0 0"/-->
-	  <origin rpy="0 1.5707 1.5707" xyz="0 0 0"/>
+	  <origin rpy="0 1.5708 1.5708" xyz="0 0 0"/>
       <geometry>
         <cylinder length="0.05" radius="0.095"/>
@@ -303,3 +307,24 @@
     </visual>
   </link>
+  <joint name = "xtion_optical_frame_joint" type="fixed">
+    <parent link="xtion_link"/>
+    <child link="xtion_optical_frame"/>
+    <origin rpy="-1.57 0 -1.57" xyz="0 0 0"/>
+  </joint>
+  <link name="xtion_optical_frame" >
+ </link>
+  <joint name = "left_optical_frame_joint" type="fixed">
+    <parent link="left_arm_camera"/>
+    <child link="left_optical_frame"/>
+    <origin rpy="0 -1.5708  0" xyz="0 0 0"/>
+  </joint>
+  <link name="left_optical_frame" >
+ </link>
+  <joint name = "right_optical_frame_joint" type="fixed">
+    <parent link="right_arm_camera"/>
+    <child link="right_optical_frame"/>
+    <origin rpy="0  -1.5708 3.14" xyz="0 0 0"/>
+  </joint>
+  <link name="right_optical_frame" >
+ </link>
 </robot>

Commit message: Name Space Remove. Grasping Moves Working

File: phoebe_description/urdf/phoebe.urdf.xacro (robot description, xacro)
@@ -32,10 +32,10 @@
   </link>
   <joint name="wheel_rear_joint" type="continuous">
+     <origin rpy="0 0 0" xyz="-0.29 0.0 0.020"/>
     <parent link="base_link"/>
     <child link="wheel_rear"/>
-    <origin rpy="0 0 0" xyz="-0.29 0.0 0.020"/>
 	<axis rpy="0 0 0" xyz="0 1 0"/>
     <limit effort="10000" velocity="1000"/>
-    <joint_properties damping="1.0" friction="1.0"/>
+    <joint_properties damping="0.0" friction="0.0"/>
   </joint>
   <link name="wheel_rear">
@@ -50,5 +50,5 @@
       <origin rpy="0 1.5707 1.5707" xyz="0 0 0"/>
       <geometry>
-        <cylinder length="0.1" radius="0.02"/>
+        <cylinder length="0.025" radius="0.02"/>
       </geometry>
       <material name="blackish">
@@ -59,5 +59,5 @@
       <origin rpy="0 1.5707 1.5707" xyz="0 0 0"/>
       <geometry>
-        <cylinder length="0.1" radius="0.02"/>
+        <cylinder length="0.025" radius="0.02"/>
       </geometry>
     </collision>
@@ -69,5 +69,5 @@
 	<axis rpy="0 0 0" xyz="0 1 0"/>
     <limit effort="10000" velocity="1000"/>
-    <joint_properties damping="1.0" friction="1.0"/>
+    <joint_properties damping="0.0" friction="0.0"/>
   </joint>
   <link name="wheel_front">
@@ -81,5 +81,5 @@
      <origin rpy="0 1.5707 1.5707" xyz="0 0 0"/>
      <geometry>
-        <cylinder length="0.1" radius="0.02"/>
+        <cylinder length="0.025" radius="0.02"/>
       </geometry>
       <material name="blackish"/>
@@ -88,5 +88,5 @@
       <origin rpy="0 1.5707 1.5707" xyz="0 0 0"/>
       <geometry>
-        <cylinder length="0.1" radius="0.02"/>
+        <cylinder length="0.025" radius="0.02"/>
       </geometry>
     </collision>
